File: hardware/vl4e3p.brd (EAGLE design)
At the start: 68 x 39 mm, 43 parts, among them Q1 AO3401A

Commit message: hardware: increase current limit of stepdown
The old resistor value was based on a very tightly calculated current
limit and was also rounded down to match an E12 value. This caused some
aging Vaporlights to fail when drawing more current (e.g. displaying all
white).
Parts:
- R33: value 15k -> 22k
Changed lines of the file:
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@@
 <?xml version="1.0" encoding="utf-8"?>
 <!DOCTYPE eagle SYSTEM "eagle.dtd">
-<eagle version="6.2">
+<eagle version="6.5.0">
 <drawing>
 <settings>
@@
 </class>
 </classes>
-<designrules>
+<designrules name="default">
 <description language="de">&lt;b&gt;EAGLE Design Rules&lt;/b&gt;
 &lt;p&gt;
@@
 <element name="U$9" library="tps40055" package="TSSOP16" value="TPS40055" x="54.61" y="13.843" smashed="yes" rot="MR270"/>
 <element name="C4" library="rcl" package="C0805" value="100p" x="51.435" y="18.923" smashed="yes" rot="MR270"/>
-<element name="R33" library="rcl" package="R0805" value="15k" x="53.467" y="18.923" smashed="yes" rot="MR90"/>
+<element name="R33" library="rcl" package="R0805" value="22k" x="53.467" y="18.923" smashed="yes" rot="MR90"/>
 <element name="C5" library="rcl" package="C0805" value="1u" x="47.625" y="18.923" smashed="yes" rot="MR270"/>
 <element name="C6" library="rcl" package="C0805" value="1u" x="45.72" y="11.557" smashed="yes" rot="MR270"/>
